File: ee/board/MPU.kicad_sch (KiCad schematic)
At the start: 7 parts, among them U10 ALLWINNER_D1, Y4 ECS-240-12-37B-CKY-TR

Commit message: Added the footprints into the design.
Parts:
- U10: footprint ALLWINNER_D1:BGA337C65P20X20_1300X1300X133 -> allwinnder_d1:BGA337C65P20X20_1300X1300X133; Availability Not in stock -> (none); Check_prices https://www.snapeda.com/parts/ALLWINNER%20D1/Allwinner+Tech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 -> (none); MANUFACTURER Allwinner Technology -> (none); MAXIMUM_PACKAGE_HEIGHT 1.33mm -> (none); MF Allwinner Technology -> (none); MP ALLWINNER D1 -> (none); PARTREV 0.1 -> (none); Package Package -> (none); Price None -> (none); STANDARD IPC 7351B -> (none); SnapEDA_Link https://www.snapeda.com/parts/ALLWINNER%20D1/Allwinner+Tech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 -> (none)
Other:
- moved on the sheet: C91, C93, U10A, U10B, U10C, U10D, U10E, U10F, U10G, XTAL1, Y4
