File: hat/nff_pcb/a33_power.kicad_sch (KiCad schematic)
At the start: 25 parts, among them U2 A33

Commit message: R0.1 Released
Parts:
- C53, C54, C55, C56, C69, C70: MPN GRM158R60J226ME01D -> GRM155R60J226ME11D
Changed lines of the file:
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@@
 			)
 		)
-		(property "MPN" "GRM158R60J226ME01D"
+		(property "MPN" "GRM155R60J226ME11D"
 			(at 95.25 100.33 0)
 			(effects
@@
 			)
 		)
-		(property "MPN" "GRM158R60J226ME01D"
+		(property "MPN" "GRM155R60J226ME11D"
 			(at 95.25 43.18 0)
 			(effects
@@
 			)
 		)
-		(property "MPN" "GRM158R60J226ME01D"
+		(property "MPN" "GRM155R60J226ME11D"
 			(at 142.24 127 0)
 			(effects
@@
 			)
 		)
-		(property "MPN" "GRM158R60J226ME01D"
+		(property "MPN" "GRM155R60J226ME11D"
 			(at 92.71 73.66 0)
 			(effects
@@
 			)
 		)
-		(property "MPN" "GRM158R60J226ME01D"
+		(property "MPN" "GRM155R60J226ME11D"
 			(at 140.97 100.33 0)
 			(effects
@@
 			)
 		)
-		(property "MPN" "GRM158R60J226ME01D"
+		(property "MPN" "GRM155R60J226ME11D"
 			(at 100.33 127 0)
 			(effects
