File: hat/nff_pcb/a33_ram.kicad_sch (KiCad schematic)
At the start: 8 parts, among them U2 A33

Commit message: R0.1 Released
Parts:
- R4, R5: MPN 4-1879208-9 -> RT0402BRD071KL
Changed lines of the file:
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@@
 			)
 		)
-		(property "MPN" "4-1879208-9"
+		(property "MPN" "RT0402BRD071KL"
 			(at 104.14 46.99 0)
 			(effects
@@
 			)
 		)
-		(property "MPN" "4-1879208-9"
+		(property "MPN" "RT0402BRD071KL"
 			(at 104.14 55.88 0)
 			(effects
