File: hat/nff_pcb/gpio.kicad_sch (KiCad schematic)
At the start: 26 parts, among them SW1 SW_Push, U10 CH340C, U13 74AHC1G32, U2 A33, Y1 24Mhz, Y2 32.768khz

Commit message: R0.1 Released
Parts:
- removed U13: 74AHC1G32, Package_TO_SOT_SMD:SOT-353_SC-70-5, symbol 74xGxx:74AHC1G32
- added R15: 100k, Resistor_SMD:R_0402_1005Metric, symbol Device:R_Small_US
- added U13: 74LVC1G08, Package_TO_SOT_SMD:SOT-353_SC-70-5, symbol 74xGxx:74LVC1G08
Connections:
- net +3V3: now also R15.2, U13.5 (VCC)
- net GND: now also U13.3 (GND)
- net UART0_TX: now also R15.1, U13.2
- net UART_TX: now also U13.4
- net at U10.2 (TXD): now also U13.1
Changed lines of the file:
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@@
 	)
 	(junction
-		(at 104.14 170.18)
+		(at 240.03 116.84)
 		(diameter 0)
 		(color 0 0 0 0)
 	)
 	(junction
-		(at 240.03 116.84)
+		(at 158.75 100.33)
 		(diameter 0)
 		(color 0 0 0 0)
 	)
 	(junction
-		(at 158.75 100.33)
+		(at 128.27 128.27)
 		(diameter 0)
 		(color 0 0 0 0)
 	)
 	(junction
-		(at 128.27 128.27)
+		(at 105.41 170.18)
 		(diameter 0)
 		(color 0 0 0 0)
@@
 	(wire
 		(pts
-			(xy 104.14 170.18) (xy 104.14 175.26)
+			(xy 105.41 170.18) (xy 105.41 175.26)
 		)
 		(stroke
@@
 	(wire
 		(pts
-			(xy 104.14 170.18) (xy 101.6 170.18)
+			(xy 101.6 170.18) (xy 105.41 170.18)
 		)
 		(stroke
@@
 	(wire
 		(pts
-			(xy 100.33 179.07) (xy 104.14 175.26)
+			(xy 101.6 179.07) (xy 105.41 175.26)
 		)
 		(stroke
@@
 	(wire
 		(pts
-			(xy 106.68 170.18) (xy 104.14 170.18)
+			(xy 106.68 170.18) (xy 105.41 170.18)
 		)
 		(stroke
@@
 	(wire
 		(pts
-			(xy 96.52 179.07) (xy 100.33 179.07)
+			(xy 96.52 179.07) (xy 101.6 179.07)
 		)
 		(stroke
@@
 	(wire
 		(pts
+			(xy 105.41 158.75) (xy 105.41 161.29)
+		)
+		(stroke
+			(width 0)
+			(type default)
+		)
+	)
+	(wire
+		(pts
 			(xy 147.32 97.79) (xy 142.24 97.79)
 		)
@@
 		)
 	)
+	(wire
+		(pts
+			(xy 105.41 166.37) (xy 105.41 170.18)
+		)
+		(stroke
+			(width 0)
+			(type default)
+		)
+	)
 	(bus
 		(pts
@@
 	)
 	(symbol
+		(lib_id "74xGxx:74LVC1G08")
+		(at 86.36 167.64 0)
+		(mirror y)
+		(unit 1)
+		(exclude_from_sim no)
+		(in_bom yes)
+		(on_board yes)
+		(dnp no)
+		(fields_autoplaced yes)
+		(property "Reference" "U13"
+			(at 89.3765 157.48 0)
+			(effects
+				(font
+					(size 1.27 1.27)
+				)
+				(justify right)
+			)
+		)
+		(property "Value" "74LVC1G08"
+			(at 89.3765 160.02 0)
+			(effects
+				(font
+					(size 1.27 1.27)
+				)
+				(justify right)
+			)
+		)
+		(property "Footprint" "Package_TO_SOT_SMD:SOT-353_SC-70-5"
+			(at 86.36 167.64 0)
+			(effects
+				(font
+					(size 1.27 1.27)
+				)
+				(hide yes)
+			)
+		)
+		(property "Datasheet" "https://www.ti.com/lit/ds/symlink/sn74lvc1g08.pdf"
+			(at 86.36 167.64 0)
+			(effects
+				(font
+					(size 1.27 1.27)
+				)
+				(hide yes)
+			)
+		)
+		(property "Description" "Single AND Gate, Low-Voltage CMOS"
+			(at 86.36 167.64 0)
+			(effects
+				(font
+					(size 1.27 1.27)
+				)
+				(hide yes)
+			)
+		)
+		(property "MPN" "SN74LVC1G08DCKR"
+			(at 86.36 167.64 0)
+			(effects
+				(font
+					(size 1.27 1.27)
+				)
+				(hide yes)
+			)
+		)
+		(pin "5"
+		)
+		(pin "3"
+		)
+		(pin "1"
+		)
+		(pin "4"
+		)
+		(pin "2"
+		)
+		(instances
+			(project ""
+				(path "/3fcdd6ae-e60a-4a06-818a-95d65ab6c907/00000000-0000-0000-0000-00006063be69"
+					(reference "U13")
+					(unit 1)
+				)
+			)
+		)
+	)
+	(symbol
 		(lib_id "Jumper:Jumper_2_Small_Open")
 		(at 93.98 179.07 0)
@@
 	)
 	(symbol
+		(lib_id "Device:R_Small_US")
+		(at 105.41 163.83 180)
+		(unit 1)
+		(exclude_from_sim no)
+		(in_bom yes)
+		(on_board yes)
+		(dnp no)
+		(property "Reference" "R15"
+			(at 108.966 162.814 0)
+			(effects
+				(font
+					(size 1.27 1.27)
+				)
+			)
+		)
+		(property "Value" "100k"
+			(at 108.966 164.592 0)
+			(effects
+				(font
+					(size 1.27 1.27)
+				)
+			)
+		)
+		(property "Footprint" "Resistor_SMD:R_0402_1005Metric"
+			(at 105.41 163.83 0)
+			(effects
+				(font
+					(size 1.27 1.27)
+				)
+				(hide yes)
+			)
+		)
+		(property "Datasheet" "~"
+			(at 105.41 163.83 0)
+			(effects
+				(font
+					(size 1.27 1.27)
+				)
+				(hide yes)
+			)
+		)
+		(property "Description" ""
+			(at 105.41 163.83 0)
+			(effects
+				(font
+					(size 1.27 1.27)
+				)
+				(hide yes)
+			)
+		)
+		(property "MPN" "RC0402FR-13100KL"
+			(at 105.41 163.83 90)
+			(effects
+				(font
+					(size 1.27 1.27)
+				)
+				(hide yes)
+			)
+		)
+		(pin "1"
+		)
+		(pin "2"
+		)
+		(instances
+			(project "hardware"
+				(path "/3fcdd6ae-e60a-4a06-818a-95d65ab6c907/00000000-0000-0000-0000-00006063be69"
+					(reference "R15")
+					(unit 1)
+				)
+			)
+		)
+	)
+	(symbol
 		(lib_id "power:+3V3")
 		(at 128.27 127 0)
@@
 	)
 	(symbol
-		(lib_id "74xGxx:74AHC1G32")
-		(at 86.36 167.64 0)
-		(mirror y)
-		(unit 1)
-		(exclude_from_sim no)
-		(in_bom yes)
-		(on_board yes)
-		(dnp no)
-		(property "Reference" "U13"
-			(at 87.122 159.512 0)
-			(effects
-				(font
-					(size 1.27 1.27)
-				)
-				(justify right)
-			)
-		)
-		(property "Value" "74AHC1G32"
-			(at 87.122 161.29 0)
-			(effects
-				(font
-					(size 1.27 1.27)
-				)
-				(justify right)
-			)
-		)
-		(property "Footprint" "Package_TO_SOT_SMD:SOT-353_SC-70-5"
-			(at 86.36 167.64 0)
-			(effects
-				(font
-					(size 1.27 1.27)
-				)
-				(hide yes)
-			)
-		)
-		(property "Datasheet" "http://www.ti.com/lit/sg/scyt129e/scyt129e.pdf"
-			(at 86.36 167.64 0)
-			(effects
-				(font
-					(size 1.27 1.27)
-				)
-				(hide yes)
-			)
-		)
-		(property "Description" "Single OR Gate, Low-Voltage CMOS"
-			(at 86.36 167.64 0)
-			(effects
-				(font
-					(size 1.27 1.27)
-				)
-				(hide yes)
-			)
-		)
-		(property "MPN" "SN74LVC1G32DCKT"
-			(at 86.36 167.64 0)
-			(effects
-				(font
-					(size 1.27 1.27)
-				)
-				(hide yes)
-			)
-		)
-		(pin "1"
-		)
-		(pin "2"
-		)
-		(pin "3"
-		)
-		(pin "4"
-		)
-		(pin "5"
-		)
-		(instances
-			(project ""
-				(path "/3fcdd6ae-e60a-4a06-818a-95d65ab6c907/00000000-0000-0000-0000-00006063be69"
-					(reference "U13")
-					(unit 1)
-				)
-			)
-		)
-	)
-	(symbol
 		(lib_id "hardware-rescue:GND-power")
 		(at 121.92 135.89 0)
@@
 					(unit 1)
 				)
+			)
+		)
+	)
+	(symbol
+		(lib_id "power:+3V3")
+		(at 105.41 158.75 0)
+		(unit 1)
+		(exclude_from_sim no)
+		(in_bom yes)
+		(on_board yes)
+		(dnp no)
+		(property "Reference" "#PWR0148"
+			(at 105.41 162.56 0)
+			(effects
+				(font
+					(size 1.27 1.27)
+				)
+				(hide yes)
+			)
+		)
+		(property "Value" "+3V3"
+			(at 105.41 154.94 0)
+			(effects
+				(font
+					(size 1.27 1.27)
+				)
+			)
+		)
+		(property "Footprint" ""
+			(at 105.41 158.75 0)
+			(effects
+				(font
+					(size 1.27 1.27)
+				)
+				(hide yes)
+			)
+		)
+		(property "Datasheet" ""
+			(at 105.41 158.75 0)
+			(effects
+				(font
+					(size 1.27 1.27)
+				)
+				(hide yes)
+			)
+		)
+		(property "Description" ""
+			(at 105.41 158.75 0)
+			(effects
+				(font
+					(size 1.27 1.27)
+				)
+				(hide yes)
+			)
+		)
+		(pin "1"
+		)
+		(instances
+			(project "hardware"
+				(path "/3fcdd6ae-e60a-4a06-818a-95d65ab6c907/00000000-0000-0000-0000-00006063be69"
+					(reference "#PWR0148")
+					(unit 1)
+				)
