File: hat/nff_pcb/hardware.kicad_sch (KiCad schematic)
At the start: 23 parts, among them J1 Micro_SD_Card_Det_Hirose_DM3AT, J2 USB_A, J3 USB_A, J4 Conn_01x08_Pin, J5 USB_C_Receptacle_USB2.0_16P, J6 Conn_01x10_Pin, U14 NUP2202, U15 NUP2202

Commit message: R0.1 Released
Parts:
- C61, C62, C94: MPN GRM158R60J226ME01D -> GRM155R60J226ME11D
Changed lines of the file:
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@@
 			)
 		)
-		(property "MPN" "GRM158R60J226ME01D"
+		(property "MPN" "GRM155R60J226ME11D"
 			(at 193.04 82.55 0)
 			(effects
@@
 			)
 		)
-		(property "MPN" "GRM158R60J226ME01D"
+		(property "MPN" "GRM155R60J226ME11D"
 			(at 245.11 106.68 0)
 			(effects
@@
 			)
 		)
-		(property "MPN" "GRM158R60J226ME01D"
+		(property "MPN" "GRM155R60J226ME11D"
 			(at 209.55 30.48 0)
 			(effects
