File: hat/nff_pcb/ram.kicad_sch (KiCad schematic)
At the start: 23 parts, among them U1 AS4C512M16D3L-12BIN

Commit message: R0.1 Released
Parts:
- R1, R2: MPN 4-1879208-9 -> RT0402BRD071KL
Changed lines of the file:
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@@
 			)
 		)
-		(property "MPN" "4-1879208-9"
+		(property "MPN" "RT0402BRD071KL"
 			(at 181.61 97.79 0)
 			(effects
@@
 			)
 		)
-		(property "MPN" "4-1879208-9"
+		(property "MPN" "RT0402BRD071KL"
 			(at 181.61 107.95 0)
 			(effects
